Commit message: added stl

File: real_color_yam/yam_plant_and_camera_mount.urdf (robot description, URDF)
Before this commit: robot yam_color, 9 links, 8 joints
Links:
- removed link link_left_finger
- removed link link_right_finger
- link link_6: geometry collision mesh filename=assets/tip.stl; visual mesh filename=assets/tip.stl
Joints:
- removed joint gripper
- removed joint gripper_mirror
